Commit message: Implement parsing and processing for inertial properties

File: industrial_payload_manager/test/urdf/payload1.xacro (robot description, xacro)
@@ -13,4 +13,9 @@
     <geometry><mesh filename="package://industrial_payload_manager/test/meshes/payload1.stl"/></geometry>
   </collision>
+  <inertial>
+    <origin xyz="0.2 0.22 0.34" rpy="0.05 0.07 0.09"/>
+    <mass value="7.232"/>
+    <inertia ixx="0.4" ixy="0.01" ixz="0.012" iyy="0.41" iyz="0.013" izz="0.31"/>
+  </inertial>
 </link>
 <link name="payload1_gripper_target"/>
